File: PrometheusII/PCB/prometheus.kicad_pcb (KiCad board)
At the start: 4 copper layers, 223.5 x 222.3 mm, 217 parts, among them J1 0878311420, J10 Conn_02x02_Odd_Even, J11 Conn_02x02_Odd_Even, J12 Conn_02x08_Odd_Even, J13 Conn_02x08_Odd_Even, J14 Conn_02x08_Odd_Even, J17 Conn_02x07_Odd_Even, J18 Conn_02x07_Odd_Even, J2 Conn_02x08_Odd_Even, J3 Conn_02x02_Odd_Even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

Commit message: output stage layout finished
Parts:
- moved TP22 0.70 mm to (141.9, 112.4)
- moved TP23 0.70 mm to (141.9, 114.0)
- moved R24 0.60 mm to (136.8, 105.6)
- moved C10 0.60 mm to (132.7, 109.3)
- moved C24 0.60 mm to (137.4, 116.0)
- moved C28 0.60 mm to (139.6, 110.4)
- moved C29 0.60 mm to (132.7, 112.6)
- moved R21 0.60 mm to (133.4, 107.0)
- moved R22 0.60 mm to (136.8, 107.1)
- moved R27 0.60 mm to (134.4, 116.0)
- moved R32 0.60 mm to (137.4, 117.4)
- moved R81 0.60 mm to (133.4, 105.6)
- moved TP21 0.60 mm to (132.7, 103.8)
- moved U4 0.60 mm to (136.1, 111.5)
- moved C15 0.30 mm to (151.1, 105.7)
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Connections:
- J11 pad 1: GND -> /OUT_P
- J11 pad 4: /OUT_P -> GND
- J4 pad 2: GND -> /OUT
- J4 pad 3: /OUT -> GND
Routing:
- net +3V3: track 647.6 -> 571.8 mm
- net GND: track 1286.1 -> 1275.1 mm, vias 80 -> 79
- net /OUT: track 34.9 -> 26.0 mm, vias 1 -> 0
- net /OUT_P: track 4.76 -> 0.00 mm
- net -12V: track 106.7 -> 108.1 mm
