File: PrometheusII/PCB/prometheus.kicad_pcb (KiCad board)
At the start: 4 copper layers, 223.5 x 222.3 mm, 240 parts, among them J1 0878311420, J10 Conn_02x02_Odd_Even, J11 Conn_02x02_Odd_Even, J12 Conn_02x08_Odd_Even, J13 Conn_02x08_Odd_Even, J14 Conn_02x08_Odd_Even, J2 Conn_02x08_Odd_Even, J3 Conn_02x02_Odd_Even, J4 Conn_02x02_Odd_Even, J7 Conn_02x08_Odd_Even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

Commit message: Some additional routing
Routing:
- net GND: track 475.3 -> 539.3 mm
- net /VOCT_CV_P: track 1.46 -> 59.9 mm, vias 0 -> 1
- net (no net): track 413.6 -> 368.4 mm
- net /PARAM_1_P: track 16.3 -> 48.1 mm
- net /VOCT_OCT_B_P: track 17.2 -> 24.7 mm
- net /VOCT_OCT_A_P: track 22.3 -> 28.2 mm
Changed lines of the file:
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@@
   (general
     (thickness 1.6)
-    (drawings 207)
-    (tracks 681)
+    (drawings 239)
+    (tracks 687)
     (zones 0)
     (modules 240)
@@
   )
   (setup
-    (last_trace_width 0.16)
+    (last_trace_width 0.15)
     (user_trace_width 0.15)
     (user_trace_width 0.1524)
@@
     (solder_mask_min_width 0.25)
     (aux_axis_origin 156.456 180.632)
-    (grid_origin 100.33 91.44)
+    (grid_origin 102.737 98.385)
     (visible_elements 7FFFFFFF)
     (pcbplotparams
@@
     )
   )
+  (gr_circle (center 102.746 98.016) (end 106.646 98.016) (layer B.SilkS) (width 0.16))
+  (gr_circle (center 102.746 98.016) (end 106.336 98.016) (layer B.SilkS) (width 0.16))
+  (gr_circle (center 102.746 98.016) (end 105.716 98.016) (layer B.SilkS) (width 0.16))
+  (gr_circle (center 102.746 98.016) (end 105.406 98.016) (layer B.SilkS) (width 0.16))
+  (gr_circle (center 102.746 98.016) (end 104.786 98.016) (layer B.SilkS) (width 0.16))
+  (gr_circle (center 102.746 98.016) (end 104.476 98.016) (layer B.SilkS) (width 0.16))
+  (gr_circle (center 95.746 99.916) (end 98.116 99.916) (layer B.SilkS) (width 0.16))
+  (gr_circle (center 95.746 99.916) (end 97.806 99.916) (layer B.SilkS) (width 0.16))
+  (gr_circle (center 95.746 99.916) (end 97.186 99.916) (layer B.SilkS) (width 0.16))
+  (gr_circle (center 95.746 99.916) (end 96.876 99.916) (layer B.SilkS) (width 0.16))
+  (gr_circle (center 79.7455 106.72) (end 82.2155 106.72) (layer B.SilkS) (width 0.16))
+  (gr_circle (center 79.7455 106.72) (end 81.9055 106.72) (layer B.SilkS) (width 0.16))
+  (gr_circle (center 79.7455 106.72) (end 81.2855 106.72) (layer B.SilkS) (width 0.16))
+  (gr_circle (center 79.7455 106.72) (end 80.9755 106.72) (layer B.SilkS) (width 0.16))
+  (gr_circle (center 70.746 104.82) (end 73.716 104.82) (layer B.SilkS) (width 0.16))
+  (gr_circle (center 70.746 104.82) (end 73.406 104.82) (layer B.SilkS) (width 0.16))
+  (gr_circle (center 70.746 104.82) (end 72.786 104.82) (layer B.SilkS) (width 0.16))
+  (gr_circle (center 70.746 104.82) (end 72.476 104.82) (layer B.SilkS) (width 0.16))
+  (gr_circle (center 63.746 106.72) (end 66.166 106.72) (layer B.SilkS) (width 0.16))
+  (gr_circle (center 63.746 106.72) (end 65.846 106.72) (layer B.SilkS) (width 0.16))
+  (gr_circle (center 63.746 106.72) (end 65.206 106.72) (layer B.SilkS) (width 0.16))
+  (gr_circle (center 63.746 106.72) (end 64.886 106.72) (layer B.SilkS) (width 0.16))
+  (gr_circle (center 47.746 111.72) (end 49.206 111.72) (layer B.SilkS) (width 0.16))
+  (gr_circle (center 47.746 111.72) (end 48.886 111.72) (layer B.SilkS) (width 0.16))
+  (gr_circle (center 102.87 93.98) (end 103.96 93.98) (layer B.SilkS) (width 0.16))
+  (gr_circle (center 100.33 93.98) (end 101.74 93.98) (layer B.SilkS) (width 0.16))
+  (gr_circle (center 100.33 93.98) (end 101.42 93.98) (layer B.SilkS) (width 0.16))
+  (gr_circle (center 70.746 99.622) (end 72.806 99.622) (layer B.SilkS) (width 0.16))
+  (gr_circle (center 70.746 99.622) (end 72.486 99.622) (layer B.SilkS) (width 0.16))
+  (gr_circle (center 54.746 99.622) (end 56.806 99.622) (layer B.SilkS) (width 0.16))
+  (gr_circle (center 54.746 99.622) (end 56.486 99.622) (layer B.SilkS) (width 0.16))
+  (gr_circle (center 47.746 97.722) (end 48.886 97.722) (layer B.SilkS) (width 0.16))
   (gr_circle (center 97.79 91.44) (end 99.2 91.44) (layer B.SilkS) (width 0.16))
   (gr_circle (center 97.79 91.44) (end 98.88 91.44) (layer B.SilkS) (width 0.16))
@@
   (segment (start 97.967637 123.071234) (end 100.467322 123.388684) (width 0.16) (layer F.Cu) (net 1))
   (segment (start 101.104803 122.572058) (end 103.281968 123.46085) (width 0.16) (layer F.Cu) (net 1))
-  (segment (start 101.225748 122.275795) (end 103.402913 123.164586) (width 0.16) (layer F.Cu) (net 0))
-  (segment (start 95.25 122.1) (end 100.33 122.1) (width 0.16) (layer F.Cu) (net 0))
+  (segment (start 101.225748 122.275795) (end 103.402913 123.164586) (width 0.16) (layer F.Cu) (net 137))
+  (segment (start 95.25 122.1) (end 100.33 122.1) (width 0.16) (layer F.Cu) (net 137))
   (segment (start 95.25 121.78) (end 100.33 121.78) (width 0.16) (layer F.Cu) (net 1))
   (segment (start 103.305905 122.795817) (end 105.684645 123.415168) (width 0.16) (layer F.Cu) (net 1))
@@
   (segment (start 104.7012 118.12235) (end 111.195685 123.639272) (width 0.16) (layer F.Cu) (net 0))
   (segment (start 104.841278 117.423098) (end 113.654003 123.576289) (width 0.16) (layer F.Cu) (net 0))
-  (segment (start 96.457735 120.49971) (end 102.047821 118.485922) (width 0.16) (layer F.Cu) (net 0))
+  (segment (start 96.457735 120.49971) (end 102.047821 118.485922) (width 0.16) (layer F.Cu) (net 138))
   (segment (start 101.939366 118.184861) (end 96.34928 120.198649) (width 0.16) (layer F.Cu) (net 0))
-  (segment (start 101.830911 117.8838) (end 96.240825 119.897589) (width 0.16) (layer F.Cu) (net 0))
+  (segment (start 101.830911 117.8838) (end 96.240825 119.897589) (width 0.16) (layer F.Cu) (net 85))
   (segment (start 101.722456 117.58274) (end 96.13237 119.596528) (width 0.16) (layer F.Cu) (net 0))
   (segment (start 95.722551 119.663758) (end 85.423992 119.451885) (width 0.16) (layer F.Cu) (net 0))
-  (segment (start 95.715969 119.983691) (end 85.41741 119.771818) (width 0.16) (layer F.Cu) (net 0))
+  (segment (start 95.715969 119.983691) (end 85.41741 119.771818) (width 0.16) (layer F.Cu) (net 85))
   (segment (start 95.709387 120.303623) (end 85.410828 120.09175) (width 0.16) (layer F.Cu) (net 0))
   (segment (start 70.283801 115.29749) (end 85.291659 119.4326) (width 0.16) (layer F.Cu) (net 0))
-  (segment (start 70.198799 115.605993) (end 85.206657 119.741104) (width 0.16) (layer F.Cu) (net 0))
+  (segment (start 70.198799 115.605993) (end 85.206657 119.741104) (width 0.16) (layer F.Cu) (net 85))
   (segment (start 70.113797 115.914497) (end 85.121655 120.049608) (width 0.16) (layer F.Cu) (net 0))
+  (segment (start 71.108775 101.323762) (end 100.557255 95.046046) (width 0.16) (layer F.Cu) (net 72))
+  (segment (start 71.175492 101.636729) (end 100.623973 95.359014) (width 0.16) (layer F.Cu) (net 1))
+  (segment (start 100.507637 95.378765) (end 103.007322 95.061315) (width 0.16) (layer F.Cu) (net 1))
+  (segment (start 103.854532 93.512244) (end 102.87 91.44) (width 0.16) (layer F.Cu) (net 1))
+  (segment (start 100.797755 94.964532) (end 102.87 93.98) (width 0.16) (layer F.Cu) (net 72))
+  (segment (start 54.152859 101.257782) (end 47.35739 98.793719) (width 0.16) (layer F.Cu) (net 72))
+  (segment (start 70.746 101.362) (end 54.746 101.362) (width 0.16) (layer F.Cu) (net 72))
+  (segment (start 70.746 101.682) (end 54.746 101.682) (width 0.16) (layer F.Cu) (net 1))
+  (segment (start 70.92179 101.674485) (end 49.858965 103.478465) (width 0.16) (layer F.Cu) (net 1))
+  (via (at 47.9043 103.5304) (size 0.6) (drill 0.3) (layers F.Cu B.Cu) (net 1))
+  (segment (start 49.858965 103.478465) (end 47.940479 103.642779) (width 0.16) (layer F.Cu) (net 1))
+  (segment (start 47.976592 103.399492) (end 54.4575 101.727) (width 0.16) (layer F.Cu) (net 1))
+  (segment (start 47.150448 98.694069) (end 45.844524 97.893976) (width 0.16) (layer F.Cu) (net 72))
+  (segment (start 45.844524 97.893976) (end 44.742 97.2185) (width 0.16) (layer B.Cu) (net 72))
+  (via (at 45.844524 97.893976) (size 0.6) (drill 0.3) (layers F.Cu B.Cu) (net 72))
   (segment (start 98.758283 90.939472) (end 100.33 93.98) (width 0.16) (layer F.Cu) (net 73))
   (segment (start 87.993158 92.290183) (end 94.963081 90.38844) (width 0.16) (layer F.Cu) (net 73))
@@
   (via (at 159.4735 98.596) (size 0.6) (drill 0.3) (layers F.Cu B.Cu) (net 1))
   (segment (start 165.33467 100.37717) (end 163.8553 100.2284) (width 0.508) (layer B.Cu) (net 1))
-  (segment (start 44.9835 98.016) (end 41.2735 98.036) (width 0.2) (layer B.Cu) (net 1))
-  (via (at 45.6535 99.456) (size 0.6) (drill 0.3) (layers F.Cu B.Cu) (net 1))
-  (segment (start 45.4335 98.106) (end 44.9835 98.016) (width 0.2) (layer B.Cu) (net 1))
   (segment (start 85.495272 101.887772) (end 87.9835 101.906) (width 0.2) (layer F.Cu) (net 1))
-  (segment (start 45.6535 99.456) (end 45.5835 98.376) (width 0.2) (layer B.Cu) (net 1))
-  (segment (start 45.5835 98.376) (end 45.4335 98.106) (width 0.2) (layer B.Cu) (net 1))
-  (segment (start 45.6535 99.456) (end 47.0535 99.546) (width 0.2) (layer F.Cu) (net 1))
-  (segment (start 41.2735 98.036) (end 40.9335 98.326) (width 0.2) (layer B.Cu) (net 1))
-  (segment (start 40.8035 99.796) (end 39.2535 102.078) (width 0.2) (layer B.Cu) (net 1))
-  (segment (start 40.9335 98.326) (end 40.8035 99.796) (width 0.2) (layer B.Cu) (net 1))
-  (segment (start 47.0535 99.546) (end 53.0035 101.976) (width 0.2) (layer F.Cu) (net 1))
   (segment (start 174.0435 110.381) (end 174.318129 110.381371) (width 0.6) (layer B.Cu) (net 1))
   (segment (start 164.8435 115.156) (end 164.8435 115.156) (width 0.6) (layer B.Cu) (net 1))
@@
   (segment (start 70.135775 93.963277) (end 63.746 92.722) (width 0.16) (layer F.Cu) (net 1))
   (segment (start 98.572716 90.267202) (end 100.33 91.44) (width 0.16) (layer F.Cu) (net 1))
+  (segment (start 47.9043 103.5304) (end 46.5835 103.759) (width 0.16) (layer B.Cu) (net 1))
   (via (at 213.4976 112.1704) (size 0.6) (drill 0.3) (layers F.Cu B.Cu) (net 2))
   (segment (start 213.4976 112.1704) (end 213.4976 114.6119) (width 0.6) (layer B.Cu) (net 2))
