File: twm/twm/twm.sch (KiCad schematic (older format))
At the start: 31 parts, among them J1 RJ45, J2 RJ45, J3 RJ45, J4 RJ45, J5 RJ45, J6 Barrel_Jack, U1 CD4504BPWR, U2 Teensy4.0_NoUnderpins

Commit message: latest version of main.py
Other:
- note added: "DNP"
Changed lines of the file:
@@
 Wire Wire Line
 	3700 1800 3700 1750
+Text Notes 6300 2800 0    50   ~ 0
+DNP
 $EndSCHEMATC
